Commit message: adjusted fingertip frame for sparseskin

File: leapXela_ss/robot.urdf (robot description, URDF)
Before this commit: robot leapXela_ss, 35 links, 34 joints
Joints:
- joint fingertip_ss_if_4_frame: origin xyz=-0 -0.025 0.0145 rpy=3.14159 -1.5708 0 -> xyz=-0.0139201 -0.025 0.0145 rpy=3.14159 -1.5708 0
- joint fingertip_ss_mf_4_frame: origin xyz=0 -0.025 0.0145 rpy=-3.14159 -1.5708 0 -> xyz=-0.0139201 -0.025 0.0145 rpy=3.14159 -1.5708 0
- joint fingertip_ss_rf_1_frame: origin xyz=-0 -0.025 0.0145 rpy=-3.14159 -1.5708 0 -> xyz=-0.0139201 -0.025 0.0145 rpy=3.14159 -1.5708 0
- joint th_fingertip_frame: origin xyz=0 -0.0300003 0.014504 rpy=3.14159 -1.5708 0 -> xyz=-0.0139201 -0.0300003 0.014504 rpy=3.14159 -1.5708 0

File: ros_ws/src/xela_description/urdf/finger.urdf (robot description, URDF)
Before this commit: robot xela_finger_generated, 5 links, 4 joints
Links:
- added link 44_ss_rf_1, mass 1e-09
- added link 44_ss_rf_2, mass 1e-09
- added link fingertip_ss_rf_1, mass 1e-09
Joints:
- added joint 44_ss_rf_1_frame: type fixed, parent rf_pip, child 44_ss_rf_1, origin xyz=-0.0113381 0.0245413 0.023 rpy=0.0 0.0 -1.5708, axis 0.0 0.0 0.0
- added joint 44_ss_rf_2_frame: type fixed, parent rf_dip, child 44_ss_rf_2, origin xyz=0.045226 0.0095 -0.0259 rpy=1.5708 0.0 3.14159, axis 0.0 0.0 0.0
- added joint fingertip_ss_rf_1_frame: type fixed, parent rf_fingertip, child fingertip_ss_rf_1, origin xyz=0.0 -0.025 0.0145 rpy=-3.14159 -1.5708 0.0, axis 0.0 0.0 0.0
- joint rf_rot: limit lower=-0.349 upper=0.349 effort=0.95 velocity=8.48 -> lower=0.349 upper=-0.349 effort=0.95 velocity=8.48

File: ros_ws/src/xela_description/urdf/thumb.urdf (robot description, URDF)
Before this commit: robot xela_thumb_generated, 5 links, 4 joints
Links:
- added link 44_ss_th_1, mass 1e-09
- added link 44_ss_th_2, mass 1e-09
- added link th_fingertip, mass 1e-09
Joints:
- added joint 44_ss_th_1_frame: type fixed, parent th_mcp, child 44_ss_th_1, origin xyz=-0.01 0.0201 0.0032 rpy=1.5708 0.0 -1.5708, axis 0.0 0.0 0.0
- added joint 44_ss_th_2_frame: type fixed, parent th_ipl, child 44_ss_th_2, origin xyz=0.01 -0.0201 0.0032 rpy=1.5708 0.0 1.5708, axis 0.0 0.0 0.0
- added joint th_fingertip_frame: type fixed, parent th_ipl, child th_fingertip, origin xyz=0.0 -0.0300003 0.014504 rpy=3.14159 -1.5708 0.0, axis 0.0 0.0 0.0
- joint th_axl: limit lower=-0.305 upper=0.436 effort=0.95 velocity=8.48 -> lower=-0.1745 upper=1.5708 effort=0.95 velocity=8.48
